File: Hardware/KiCad/GPBH.kicad_sch (KiCad schematic)
At the start: 0 parts

Commit message: Circuit Schematic Rev 1.0
First revision of the electronic circuit with all intended functionality but generic components and no footprints.
Parts:
- added C1: 47u, symbol Device:C_Polarized
- added D1, D2, D3: LED, symbol Device:LED
- added J1: 9VDC, symbol Connector:Jack-DC
- added J2: User_Pot_2, symbol Connector:Conn_01x03_Female
- added J3: User_Pot_3, symbol Connector:Conn_01x03_Female
- added J4: User_Pot_1, symbol Connector:Conn_01x03_Female
- added J5: User_EP_1, symbol Connector:Conn_01x02_Female
- added J6: Audio_In, symbol Connector:AudioJack2
- added J7: User_EP_2, symbol Connector:Conn_01x02_Female
- added J8: User_Effect, symbol Connector:Conn_01x02_Female
- added J9: Audio_Out, symbol Connector:AudioJack2
- added R1, R2, R3: 1k, symbol Device:R
- added RV1, RV2, RV3, RV4: 100k, symbol Device:R_Potentiometer
- added SW1, SW2: 3PDT_Switch, symbol GPBH:3PDT_Switch
Connections:
- new net: J5.1 (Pin_1), SW1.2 (P1)
- new net: J5.2 (Pin_2), SW1.5 (P2)
- new net: D2.1 (K), R2.1
- new net: D2.2 (A), SW1.7 (P3T1)
- new net: J9.S, RV4.2
- new net: J3.1 (Pin_1), RV3.1
- new net: J3.2 (Pin_2), RV3.2
- new net: J3.3 (Pin_3), RV3.3
- new net: J4.1 (Pin_1), RV1.1
- new net: J4.2 (Pin_2), RV1.2
- new net: J4.3 (Pin_3), RV1.3
- new net: J7.1 (Pin_1), SW1.1 (P1T1)
- new net: SW1.3 (P1T2), SW1.6 (P2T2)
- new net: J7.2 (Pin_2), SW1.4 (P2T1)
- new net: D3.1 (K), R3.1
- new net: D1.1 (K), R1.1
- new net: J2.1 (Pin_1), RV2.1
- new net: J2.2 (Pin_2), RV2.2
- new net: J2.3 (Pin_3), RV2.3
- new net: J8.1 (Pin_1), SW2.1 (P1T1)
- new net: J6.S, SW2.2 (P1)
- new net: SW2.3 (P1T2), SW2.6 (P2T2)
- new net: J8.2 (Pin_2), SW2.4 (P2T1)
- new net: D3.2 (A), SW2.7 (P3T1)
- new net +9V: C1.1, D1.2 (A), J1.2, SW1.8 (P3), SW2.8 (P3)
- new net GND: C1.2, J1.1, J6.T, J9.T, R1.2, R2.2, R3.2, RV4.3
- new net PedalOut: RV4.1, SW2.5 (P2)
- no-connect marks 0 -> 2
Other:
- note added: "Bypass Switch"
- note added: "Logarithmic Taper Potentiometer"
- note added: "Power In"
- note added: "User Accessible Potentiometers"
- note added: "User Accessible Switch"
- note added: "Volume Control"

Commit message: Schematic Rev 1.1
Added footprint and 3D model for the 6.3mm audio jack inteded to be used
and modified the schematic to use this, along with removal of the power
supply filtering to ensure that this isn't forgotten when prototyping.
Parts:
- removed C1: 47u, symbol Device:C_Polarized
- removed J6: Audio_In, symbol Connector:AudioJack2
- removed J9: Audio_Out, symbol Connector:AudioJack2
- added J3: Audio_In, GPBH:6.3mmJack, symbol Connector:AudioJack2_Switch
- added J4: Audio_Out, GPBH:6.3mmJack, symbol Connector:AudioJack2_Switch
- SW1: renamed from SW2; footprint (none) -> GPBH:Gorva-3PDT
- SW2: renamed from SW1; footprint (none) -> GPBH:Gorva-3PDT
- renumbered D3 to D2, D2 to D3, J8 to J1, J1 to J2, J4 to J5, J5 to J6, J2 to J8, J3 to J9, R3 to R2, R2 to R3, RV4 to RV1, RV1 to RV2, RV2 to RV3, RV3 to RV4
Connections:
- net GND: now also J3.T, J4.T
- net at RV1.2: now also J4.S
- net at SW1.2 (P1): now also J3.S
- no-connect marks 2 -> 6
